File: sensor.brd (EAGLE design)
At the start: 100 x 80 mm, 8 parts

Commit message: Add files via upload
Parts:
- removed C1: (no value), rcl:C050-030X075
- removed JP1: (no value), pinhead:2X03
- removed JP2, JP3: (no value), pinhead:1X04
- removed JP4: (no value), pinhead:2X04
- removed S1: (no value), switch-omron:B3F-10XX
- removed U$1: ESP32DEVKITV1, esp32-devkitv1:ESP32-DEVKITV1
- removed X1: (no value), con-ptr500:AK300/2
- added D1, D2, D3, D4, D5, D6, D7, D8: PhotoDioda, opto-trans-siemens:SFH225
- added LED1, LED2, LED3, LED4, LED5, LED6, LED7, LED8: LED putih SB, led:LED5MM
- added R1, R2, R3, R4, R5, R6, R7, R8: (no value), resistor:0207/10
- added R10, R11, R12, R13, R14, R15, R16, R9: 330, resistor:0207/10
- added SV1: (no value), con-lstb:MA10-1
Connections:
- removed net MOISTURE: JP1.2, U$1.D2
- removed net OUT1: JP2.1, U$1.D33
- removed net OUT2: JP2.2, U$1.D32
- removed net OUT3: JP2.3, U$1.D35
- removed net PH: JP1.1, U$1.D15
- removed net SCL: JP3.2, U$1.D22
- removed net SCL2: JP4.5, JP4.6, U$1.D25
- removed net SDA: JP3.1, U$1.D21
- removed net SDA2: JP4.7, JP4.8, U$1.D26
- removed net V: C1.2, JP1.3, JP1.4, JP3.3, JP4.1, JP4.2, S1.1, S1.2, U$1.3V3, U$1.D36
- removed net VIN: U$1.VIN, X1.2
- new net N$1: LED7.A, R10.1
- new net N$10: LED6.A, R11.1
- new net N$11: LED5.A, R12.1
- new net N$12: LED4.A, R13.1
- new net N$13: LED3.A, R14.1
- new net N$14: LED2.A, R15.1
- new net N$15: LED1.A, R16.1
- new net N$16: LED8.A, R9.1
- new net N$2: D7.K, R7.1, SV1.2
- new net N$3: D8.K, R8.1, SV1.1
- new net N$4: D1.K, R1.1, SV1.8
- new net N$5: D2.K, R2.1, SV1.7
- new net N$6: D3.K, R3.1, SV1.6
- new net N$7: D5.K, R5.1, SV1.4
- new net N$8: D4.K, R4.1, SV1.5
- new net N$9: D6.K, R6.1, SV1.3
- new net VCC: R1.2, R10.2, R11.2, R12.2, R13.2, R14.2, R15.2, R16.2, R2.2, R3.2, R4.2, R5.2, R6.2, R7.2, R8.2, R9.2, SV1.9
- net GND: now also D1.A, D2.A, D3.A, D4.A, D5.A, D6.A, D7.A, D8.A, LED1.K, LED2.K, LED3.K, LED4.K, LED5.K, LED6.K, LED7.K, LED8.K, SV1.10; no longer C1.1, JP1.5, JP1.6, JP2.4, JP3.4, JP4.3, JP4.4, S1.3, S1.4, U$1.GND@1, U$1.GND@2, X1.1
Routing:
- net SCL2: track 192.4 -> 0.00 mm
- net VCC: track 0.00 -> 169.5 mm
- net SDA2: track 161.0 -> 0.00 mm
- net N$3: track 0.00 -> 141.6 mm
- net V: track 124.6 -> 0.00 mm
- net N$6: track 0.00 -> 101.6 mm
- net N$4: track 0.00 -> 92.1 mm
- net N$7: track 0.00 -> 75.5 mm
- net OUT1: track 74.3 -> 0.00 mm
- net N$2: track 0.00 -> 74.3 mm
- net N$5: track 0.00 -> 70.9 mm
- net OUT2: track 68.3 -> 0.00 mm
- net OUT3: track 62.6 -> 0.00 mm
- net N$9: track 0.00 -> 45.0 mm
- net GND: track 214.9 -> 255.4 mm
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- added copper zone on layer 16, net GND
Other:
- board text added: "Umar"
- board text removed: "UmarKhtam"
